File: doc/schematics/PDCViewer.sch (EAGLE design)
At the start: 59 parts, among them IC1 MEGA8-P, IC2 MCP2515-E/P, IC3 MCP2551P, IC4 78L05, T1 BC337, T2 BC337, X1 CAN

Commit message: update schematics
- introduce connectors between controller and status LEDs
Parts:
- added JP1: (no value), pinhead:PINHD-1X10
- added JP2: (no value), pinhead:PINHD-1X10/90
- added JP3: (no value), pinhead:PINHD-1X5
- added JP4: (no value), pinhead:PINHD-1X5/90
Connections:
- new net N$24: JP2.1, R5.1
- new net N$25: JP2.2, R6.1
- new net N$26: JP2.3, R7.1
- new net N$27: JP2.4, R8.1
- new net N$28: JP2.5, R9.1
- new net N$29: JP2.6, R10.1
- new net N$30: JP2.7, R11.1
- new net N$31: JP2.8, R12.1
- new net N$32: JP2.9, R13.1
- new net N$34: JP2.10, R14.1
- new net N$35: JP4.3, R15.1
- new net N$36: JP4.2, R4.1
- new net N$37: JP4.1, R2.1
- net CS_LED1: now also JP3.1; no longer R2.1
- net CS_LED2: now also JP3.2; no longer R4.1
- net GND: now also JP3.5, JP4.5
- net LED1: now also JP1.1; no longer R5.1
- net LED10: now also JP1.10; no longer R14.1
- net LED2: now also JP1.2; no longer R6.1
- net LED3: now also JP1.3; no longer R7.1
- net LED4: now also JP1.4; no longer R8.1
- net LED5: now also JP1.5; no longer R9.1
- net LED6: now also JP1.6; no longer R10.1
- net LED7: now also JP1.7; no longer R11.1
- net LED8: now also JP1.8; no longer R12.1
- net LED9: now also JP1.9; no longer R13.1
- net N$5: now also R3.1; no longer R3.2
- net N$6: now also R3.2; no longer R3.1
- net STATUS_LED: now also JP3.3; no longer R15.1
Other:
- moved on the sheet: LED21, R10, R11, R12, R13, R14, R15, R2, R3, R4, R5, R6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
